Commit message: add sensors;

File: armsrov_description/urdf/base.xacro (robot description, xacro)
@@ -27,5 +27,5 @@
   this geometry as simple as possible to improve the performance the physics engine
   regarding the computation of collision forces) -->
-  <xacro:property name="collision_mesh_file" value="file://$(find armsrov_description)/meshes/ARMsROV_collision.stl"/>
+  <xacro:property name="collision_mesh_file" value="file://$(find armsrov_description)/meshes/ARMsROV_no_props.dae"/>
   <!-- Vehicle macro -->
   <xacro:macro name="armsrov_base" params="namespace *gazebo">
@@ -65,5 +65,5 @@
     <xacro:include filename="$(find armsrov_description)/urdf/actuators.xacro"/>
     <!-- Include the sensor modules -->
-    <!-- <xacro:include filename="$(find armsrov_description)/urdf/sensors.xacro"/> -->
+    <xacro:include filename="$(find armsrov_description)/urdf/sensors.xacro"/>
   </xacro:macro>
 </robot>

File: armsrov_description/urdf/gazebo.xacro (robot description, xacro)
@@ -4,5 +4,5 @@
     <xacro:property name="armsrov_cob" value="0 0 0.15"/>
     <!-- Vehicle's actual volume (Gazebo cannot compute the volume out of the mesh) -->
-    <xacro:property name="armsrov_volume" value="0.01390"/>
+    <xacro:property name="armsrov_volume" value="0.01370"/>
     <!-- Describing the dimensions of the vehicle's bounding box -->
     <xacro:property name="armsrov_length" value="0.40"/>

File: armsrov_description/urdf/sensors.xacro (robot description, xacro)
@@ -8,22 +8,22 @@
   -->
   <!-- Mount a GPS. -->
-  <xacro:default_gps namespace="${namespace}" parent_link="${namespace}/base_link" />
+  <!-- <xacro:default_gps namespace="${namespace}" parent_link="${namespace}/base_link" /> -->
   <!-- Mount a Pose 3D sensor. -->
-  <xacro:default_pose_3d namespace="${namespace}" parent_link="${namespace}/base_link" />
+  <!-- <xacro:default_pose_3d namespace="${namespace}" parent_link="${namespace}/base_link" /> -->
   <!-- Forward-looking sonar sensor -->
-  <xacro:forward_multibeam_p900 namespace="${namespace}" parent_link="${namespace}/base_link">
+  <!-- <xacro:forward_multibeam_p900 namespace="${namespace}" parent_link="${namespace}/base_link">
     <origin xyz="0 0 0" rpy="0 0 0"/>
-  </xacro:forward_multibeam_p900>
+  </xacro:forward_multibeam_p900> -->
   <!-- DVL  -->
-  <xacro:default_dvl namespace="${namespace}" parent_link="${namespace}/base_link">
+  <!-- <xacro:default_dvl namespace="${namespace}" parent_link="${namespace}/base_link">
     <origin xyz="0 0 0" rpy="0 0 0"/>
-  </xacro:default_dvl>
+  </xacro:default_dvl> -->
   <!-- RPT  -->
-  <xacro:default_rpt namespace="${namespace}" parent_link="${namespace}/base_link">
+  <!-- <xacro:default_rpt namespace="${namespace}" parent_link="${namespace}/base_link">
     <origin xyz="0 0 0" rpy="0 0 0"/>
-  </xacro:default_rpt>
+  </xacro:default_rpt> -->
   <!-- Pressure  -->
   <xacro:default_pressure namespace="${namespace}" parent_link="${namespace}/base_link">
-    <origin xyz="0 0 0" rpy="0 0 0"/>
+    <origin xyz="-0.1 0 0" rpy="0 0 0"/>
   </xacro:default_pressure>
   <!-- IMU  -->
@@ -32,6 +32,6 @@
   </xacro:default_imu>
   <!-- Mount a camera  -->
-  <xacro:default_camera namespace="${namespace}" parent_link="${namespace}/base_link" suffix="">
-    <origin xyz="0 0 0" rpy="0 0 0"/>
-  </xacro:default_camera>
+  <!-- <xacro:default_camera namespace="${namespace}" parent_link="${namespace}/base_link" suffix="">
+    <origin xyz="0.1 0.1 -0.1" rpy="0 0 0"/>
+  </xacro:default_camera> -->
 </robot>

Commit message: change cob and cog;

File: armsrov_description/urdf/base.xacro (robot description, xacro)
@@ -14,5 +14,5 @@
   <xacro:property name="mass" value="13.64"/>
   <!-- Center of gravity -->
-  <xacro:property name="cog" value="0 0 0"/>
+  <xacro:property name="cog" value="0 0 -0.1"/>
   <!-- Fluid density -->
   <xacro:property name="rho" value="1028"/>

File: armsrov_description/urdf/gazebo.xacro (robot description, xacro)
@@ -2,5 +2,5 @@
 <robot xmlns:xacro="http://www.ros.org/wiki/xacro">
     <!-- Center of buoyancy -->
-    <xacro:property name="armsrov_cob" value="0 0 0.15"/>
+    <xacro:property name="armsrov_cob" value="0 0 0.20"/>
     <!-- Vehicle's actual volume (Gazebo cannot compute the volume out of the mesh) -->
     <xacro:property name="armsrov_volume" value="0.01370"/>
